Commit message: add gnssnav

File: simulator/vehicle/xacro/parts/active_caster_macro.xacro (robot description, xacro)
@@ -27,5 +27,5 @@
     <link name="${caster_back}_link">
       <visual>
-        <origin xyz="${x} ${y} ${z}" rpy="${roll} ${pitch} ${yaw+PI/2}"/>
+        <origin xyz="${x} ${y} ${z}" rpy="${roll} ${pitch} ${yaw}"/>
         <geometry>
           <mesh filename="${MESH_FILE}" scale="${SCALE} ${SCALE} ${SCALE}"/>
@@ -33,5 +33,5 @@
       </visual>
       <collision>
-        <origin xyz="${x} ${y} ${z}" rpy="${roll} ${pitch} ${yaw+PI/2}"/>
+        <origin xyz="${x} ${y} ${z}" rpy="${roll} ${pitch} ${yaw}"/>
         <geometry>
           <mesh filename="${MESH_FILE}" scale="${SCALE} ${SCALE} ${SCALE}"/>
@@ -43,5 +43,5 @@
       </collision>
       <inertial>
-        <origin xyz="${x} ${y} ${z}" rpy="${roll} ${pitch} ${yaw+PI/2}"/>
+        <origin xyz="${x} ${y} ${z}" rpy="${roll} ${pitch} ${yaw}"/>
         <mass value="0.005" />
         <inertia ixx="0.001" ixy="0.0" ixz="0.0" iyy="0.001" iyz="0.0" izz="0.001"/>

File: simulator/vehicle/xacro/parts/caster_trail_macro.xacro (robot description, xacro)
@@ -26,5 +26,5 @@
     <link name="${caster_back}_link">
       <visual>
-        <origin xyz="${x} ${y} ${z}" rpy="${roll} ${pitch} ${yaw+PI/2}"/>
+        <origin xyz="${x} ${y} ${z}" rpy="${roll} ${pitch} ${yaw}"/>
         <geometry>
           <mesh filename="${MESH_FILE}" scale="${SCALE} ${SCALE} ${SCALE}"/>
@@ -32,5 +32,5 @@
       </visual>
       <collision>
-        <origin xyz="${x} ${y} ${z}" rpy="${roll} ${pitch} ${yaw+PI/2}"/>
+        <origin xyz="${x} ${y} ${z}" rpy="${roll} ${pitch} ${yaw}"/>
         <geometry>
           <mesh filename="${MESH_FILE}" scale="${SCALE} ${SCALE} ${SCALE}"/>
@@ -42,5 +42,5 @@
       </collision>
       <inertial>
-        <origin xyz="${x} ${y} ${z}" rpy="${roll} ${pitch} ${yaw+PI/2}"/>
+        <origin xyz="${x} ${y} ${z}" rpy="${roll} ${pitch} ${yaw}"/>
         <mass value="0.005" />
         <inertia ixx="0.001" ixy="0.0" ixz="0.0" iyy="0.001" iyz="0.0" izz="0.001"/>
