Commit message: ✨feat: カメラ座標系link定義

File: simulator/models/ai_car1/model.urdf (robot description, URDF)
Before this commit: robot ai_car1, 11 links, 10 joints
Links:
- added link camera_optical_link
Joints:
- added joint camera_optical_joint: type fixed, parent camera_link, child camera_optical_link, origin xyz=0 0 0 rpy=-1.5707963267948966 0 -1.5707963267948966
