Commit message: feat: simのカメラと車両寸法を実機に合わせる

File: simulator/models/ai_car1/model.urdf (robot description, URDF)
Before this commit: robot ai_car1, 11 links, 10 joints
Links:
- link caster: geometry collision sphere radius=0.125; visual sphere radius=0.125
- link left_wheel: geometry collision mesh filename=package://simulator/models/ai_car1/meshes/tire.dae scale=0.0625 0.127 0.127; visual mesh filename=package://simulator/models/ai_car1/meshes/tire.dae scale=0.0625 0.127 0.127
- link right_wheel: geometry collision mesh filename=package://simulator/models/ai_car1/meshes/tire.dae scale=0.0625 0.127 0.127; visual mesh filename=package://simulator/models/ai_car1/meshes/tire.dae scale=0.0625 0.127 0.127
Joints:
- joint base_to_chassis: origin xyz=0 0 0.15 rpy=0 0 0 -> xyz=0 0 0.127 rpy=0 0 0
- joint camera_joint: origin xyz=0.055 0 0.54 rpy=-0.0034939840 0.0436329672 -0.0036430636 -> xyz=-0.008 0.0325 0.4277 rpy=0.00867605 -0.00346759 0.00624156
- joint caster_pitch_joint: origin xyz=0 0 0 rpy=0 0 0 -> xyz=0 0.04 0 rpy=0 0 0
- joint caster_yaw_wheel: origin xyz=-0.8 0 0 rpy=0 0 1.57 -> xyz=-0.733 0 -0.002 rpy=0 0 1.57
